File: ESPxx Programmer/ESPxx Programmer.kicad_pcb (KiCad board)
At the start: 2 copper layers, 83.8 x 47.6 mm, 12 parts, among them J1 FTDI Programmer, SW1 Flash, SW2 Reset, U1 ESP32-CAM, U2 ESP-01h, U3 AMS1117-3.3, U4 Level shifter BSS138

Commit message: page settings
Other:
- board text added: "${TITLE}-${REVISION} Design: Jon Sagebrand github.com/jonsag/miscPCBs"
- board text removed: "ESPxxProgrammer Design: Jon Sagebrand github.com/jonsag/miscPCBs"
Changed lines of the file:
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@@
   )
   (paper "A4")
+  (title_block
+    (title "ESPxx Programmer")
+    (date "2022-10-23")
+    (rev "0.1")
+  )
   (layers
     (0 "F.Cu" signal)
@@
   (gr_line (start 153.035 54.61) (end 153.035 102.235) (layer "Edge.Cuts") (width 0.1))
   (gr_line (start 69.215 102.235) (end 69.215 54.61) (layer "Edge.Cuts") (width 0.1))
-  (gr_text "ESPxxProgrammer\nDesign: Jon Sagebrand\ngithub.com/jonsag/miscPCBs" (at 140.97 97.155) (layer "B.Cu")
+  (gr_text "${TITLE}-${REVISION}\nDesign: Jon Sagebrand\ngithub.com/jonsag/miscPCBs" (at 140.97 97.155) (layer "B.Cu")
     (effects (font (size 1.27 1.27) (thickness 0.254)) (justify left mirror))
   )
