File: ESPxx Programmer/ESPxx Programmer.kicad_sch (KiCad schematic)
At the start: 12 parts, among them J1 FTDI Programmer, SW1 Flash, SW2 Reset, U1 ESP32-CAM, U2 ESP-01h, U3 AMS1117-3.3, U4 Level shifter BSS138

Commit message: page settings
Other:
- title: (none) -> ESPxx Programmer
Changed lines of the file:
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@@
 (kicad_sch (version 20211123) (generator eeschema)
   (paper "A4")
+  (title_block
+    (title "ESPxx Programmer")
+    (date "2022-10-23")
+    (rev "0.1")
+  )
   (junction (at 170.18 85.09) (diameter 0) (color 0 0 0 0)
   )
